File: pcb/kicad_files/neodox.kicad_pcb (KiCad board)
At the start: 2 copper layers, 163.9 x 129.1 mm, 78 parts, among them J1 Conn_01x02_Female, K0 KEYSW, K1 KEYSW, K10 KEYSW, K11 KEYSW, K12 KEYSW, K13 KEYSW, K14 KEYSW, K15 KEYSW, K16 KEYSW, K2 KEYSW, K20 KEYSW, K21 KEYSW, K22 KEYSW, K23 KEYSW, K24 KEYSW, K25 KEYSW, K26 KEYSW, K3 KEYSW, K30 KEYSW, K31 KEYSW, K32 KEYSW, K33 KEYSW, K34 KEYSW, K35 KEYSW, K36 KEYSW, K4 KEYSW, K40 KEYSW, K41 KEYSW, K42 KEYSW, K43 KEYSW, K44 KEYSW, K45 KEYSW, K46 KEYSW, K5 KEYSW, K6 KEYSW, SW1 SW_DPDT_x2, U1 ProMicro

Commit message: chchchchangeees
Parts:
- removed D0, D36, D40, D41, D42, D43, D44, D45, D46: D, keyboard_reversible:Diode-dual
- removed K0, K1, K10, K11, K12, K13, K14, K15, K16, K2, K20, K21, K22, K23, K24, K25, K26, K3, K30, K31, K32, K33, K34, K35, K36, K4, K40, K41, K42, K43, K44, K45, K46, K5, K6: KEYSW, Keyboard_reversible:Kailh_socket_MX_optional_reversible
- added D17: D, Keyboard_reversible:Diode-dual, F.Cu at (94.2, 83.7)
- added D18: D, Keyboard_reversible:Diode-dual, F.Cu at (113.1, 81.3)
- added D19: D, Keyboard_reversible:Diode-dual, F.Cu at (132.5, 83.7)
- added D27: D, Keyboard_reversible:Diode-dual, F.Cu at (151.3, 104.9)
- added D28: D, Keyboard_reversible:Diode-dual, F.Cu at (187.0, 119.7)
- added D29: D, Keyboard_reversible:Diode-dual, F.Cu at (56.2, 126.4)
- added D7: D, Keyboard_reversible:Diode-dual, F.Cu at (169.9, 56.6)
- added D8: D, Keyboard_reversible:Diode-dual, F.Cu at (57.1, 69.6)
- added D9: D, Keyboard_reversible:Diode-dual, F.Cu at (75.3, 69.4)
- added H1: MountingHole, MountingHole:MountingHole_3.2mm_M3, F.Cu at (160.7, 49.2)
- added H2: MountingHole, MountingHole:MountingHole_3.2mm_M3, F.Cu at (65.7, 108.6)
- added H3: MountingHole, MountingHole:MountingHole_3.2mm_M3, F.Cu at (65.7, 51.6)
- added H4: MountingHole, MountingHole:MountingHole_3.2mm_M3, F.Cu at (175.6, 119.8)
- added S1: KEYSW, Keyboard_reversible:Kailh_socket_MX_optional_reversible, F.Cu at (56.2, 42.1)
- added S10: KEYSW, Keyboard_reversible:Kailh_socket_MX_optional_reversible, F.Cu at (94.2, 56.3)
- added S11: KEYSW, Keyboard_reversible:Kailh_socket_MX_optional_reversible, F.Cu at (113.2, 53.9)
- added S12: KEYSW, Keyboard_reversible:Kailh_socket_MX_optional_reversible, F.Cu at (132.2, 56.3)
- added S13: KEYSW, Keyboard_reversible:Kailh_socket_MX_optional_reversible, F.Cu at (151.2, 58.7)
- added S14: KEYSW, Keyboard_reversible:Kailh_socket_MX_optional_reversible, F.Cu at (170.2, 72.0)
- added S15: KEYSW, Keyboard_reversible:Kailh_socket_MX_optional_reversible, F.Cu at (56.2, 80.1)
- added S16: KEYSW, Keyboard_reversible:Kailh_socket_MX_optional_reversible, F.Cu at (75.2, 80.1)
- added S17: KEYSW, Keyboard_reversible:Kailh_socket_MX_optional_reversible, F.Cu at (94.2, 75.3)
- added S18: KEYSW, Keyboard_reversible:Kailh_socket_MX_optional_reversible, F.Cu at (113.2, 72.9)
- added S19: KEYSW, Keyboard_reversible:Kailh_socket_MX_optional_reversible, F.Cu at (132.2, 75.3)
- added S2: KEYSW, Keyboard_reversible:Kailh_socket_MX_optional_reversible, F.Cu at (75.2, 42.1)
- added S20: KEYSW, Keyboard_reversible:Kailh_socket_MX_optional_reversible, F.Cu at (151.2, 77.7)
- added S21: KEYSW, Keyboard_reversible:Kailh_socket_MX_optional_reversible, F.Cu at (174.5, 102.8)
- added S22: KEYSW, Keyboard_reversible:Kailh_socket_MX_optional_reversible, F.Cu at (56.2, 99.1)
- added S23: KEYSW, Keyboard_reversible:Kailh_socket_MX_optional_reversible, F.Cu at (75.2, 99.1)
- added S24: KEYSW, Keyboard_reversible:Kailh_socket_MX_optional_reversible, F.Cu at (94.2, 94.3)
- added S25: KEYSW, Keyboard_reversible:Kailh_socket_MX_optional_reversible, F.Cu at (113.2, 92.0)
- added S26: KEYSW, Keyboard_reversible:Kailh_socket_MX_optional_reversible, F.Cu at (132.2, 94.4)
- added S27: KEYSW, Keyboard_reversible:Kailh_socket_MX_optional_reversible, F.Cu at (151.2, 96.7)
- added S28: KEYSW, Keyboard_reversible:Kailh_socket_MX_optional_reversible, F.Cu at (191.0, 112.3)
- added S29: KEYSW, Keyboard_reversible:Kailh_socket_MX_optional_reversible, F.Cu at (56.2, 118.1)
- added S3: KEYSW, Keyboard_reversible:Kailh_socket_MX_optional_reversible, F.Cu at (94.2, 37.3)
- added S30: KEYSW, Keyboard_reversible:Kailh_socket_MX_optional_reversible, F.Cu at (75.2, 118.1)
- added S31: KEYSW, Keyboard_reversible:Kailh_socket_MX_optional_reversible, F.Cu at (94.2, 113.3)
- added S32: KEYSW, Keyboard_reversible:Kailh_socket_MX_optional_reversible, F.Cu at (113.2, 111.0)
- added S33: KEYSW, Keyboard_reversible:Kailh_socket_MX_optional_reversible, F.Cu at (137.9, 117.1)
- added S34: KEYSW, Keyboard_reversible:Kailh_socket_MX_optional_reversible, F.Cu at (162.5, 123.3)
- added S35: KEYSW, Keyboard_reversible:Kailh_socket_MX_optional_reversible, F.Cu at (179.0, 132.8)
- added S4: KEYSW, Keyboard_reversible:Kailh_socket_MX_optional_reversible, F.Cu at (113.2, 34.9)
- added S5: KEYSW, Keyboard_reversible:Kailh_socket_MX_optional_reversible, F.Cu at (132.2, 37.3)
- added S6: KEYSW, Keyboard_reversible:Kailh_socket_MX_optional_reversible, F.Cu at (151.2, 39.7)
- added S7: KEYSW, Keyboard_reversible:Kailh_socket_MX_optional_reversible, F.Cu at (170.2, 48.2)
- added S8: KEYSW, Keyboard_reversible:Kailh_socket_MX_optional_reversible, F.Cu at (56.2, 61.1)
- added S9: KEYSW, Keyboard_reversible:Kailh_socket_MX_optional_reversible, F.Cu at (75.2, 61.1)
- D1, D10, D11, D12, D13, D14, D15, D16, D2, D20, D21, D22, D23, D24, D25, D26, D3, D30, D31, D32, D33, D34, D35, D4, D5, D6: footprint keyboard_reversible:Diode-dual -> Keyboard_reversible:Diode-dual
- U1: footprint keyboard_reversible:ProMicro -> Keyboard_reversible:ProMicro_unrouted
- moved D15 107.7 mm to (56.2, 88.3)
- moved D16 105.3 mm to (74.9, 88.4)
- moved D21 88.5 mm to (170.5, 110.2), turned to 150 degrees
- moved D20 85.0 mm to (151.1, 86.1)
- moved D23 55.6 mm to (75.2, 107.6)
- moved D22 54.3 mm to (56.1, 107.5)
- moved D24 52.1 mm to (94.3, 102.6)
- moved D25 50.8 mm to (113.3, 100.5)
- moved D26 48.0 mm to (132.1, 102.9), turned to 180 degrees
- moved D35 36.0 mm to (171.2, 137.9), turned to 150 degrees
- moved D14 33.4 mm to (170.9, 80.5)
- moved D6 30.1 mm to (151.2, 48.2)
- moved D2 29.9 mm to (75.0, 50.7)
- moved D34 29.8 mm to (154.6, 128.4), turned to 150 degrees
- moved D3 29.4 mm to (94.1, 45.7)
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Connections:
- D15 pad 1: row1 -> row2
- D16 pad 1: row1 -> row2
- D22 pad 1: row2 -> row3
- D23 pad 1: row2 -> row3
- D24 pad 1: row2 -> row3
- D25 pad 1: row2 -> row3
- D26 pad 1: row2 -> row3
- D30 pad 1: row3 -> row4
- D31 pad 1: row3 -> row4
- D32 pad 1: row3 -> row4
- D33 pad 1: row3 -> row4
- D34 pad 1: row3 -> row4
- D35 pad 1: row3 -> row4
Routing:
- net col0: track 0.00 -> 344.4 mm, vias 0 -> 1
- net col1: track 0.00 -> 291.7 mm, vias 0 -> 1
- net col2: track 0.00 -> 267.8 mm, vias 0 -> 2
- net row4: track 0.00 -> 253.4 mm, vias 0 -> 1
- net col4: track 0.00 -> 248.2 mm, vias 0 -> 3
- net col3: track 0.00 -> 248.0 mm, vias 0 -> 2
- net row3: track 0.00 -> 228.6 mm, vias 0 -> 1
- net col5: track 0.00 -> 222.1 mm, vias 0 -> 3
- net row2: track 0.00 -> 214.6 mm, vias 0 -> 1
- net col6: track 0.00 -> 198.1 mm, vias 0 -> 2
- net row1: track 0.00 -> 188.9 mm, vias 0 -> 1
- net row0: track 0.00 -> 181.8 mm, vias 0 -> 1
- net VCC: track 0.00 -> 88.7 mm, vias 0 -> 1
- net SDA: track 0.00 -> 54.2 mm, vias 0 -> 1
- net rgb_data: track 0.00 -> 52.4 mm, vias 0 -> 2
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- added copper zone on B.Cu, net GND
- added copper zone on F.Cu, net GND
Other:
- board text added: "NEODOX"
