File: pcb/kicad_files/neodox_pre_routing.kicad_pcb (KiCad board)
At the start: 2 copper layers, 163.9 x 129.1 mm, 82 parts, among them J1 Conn_01x02_Female, SW1 SW_DPDT_x2, U1 ProMicro

Commit message: Change name
Other:
- board text added: "neo-redox"
- board text removed: "NEODOX"
